File: GOATS/_saved_GOATS.sch (KiCad schematic (older format))
At the start: 56 parts, among them J1 TERM_BLOCK, J10 Conn_01x01, J11 Conn_01x01, J12 Conn_01x01, J13 TERM_BLOCK, J2 TERM_BLOCK, J3 TERM_BLOCK, J4 TERM_BLOCK, J5 TERM_BLOCK, J6 TERM_BLOCK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

Commit message: KiCAD Proj. With Layout
Parts:
- gave numbers to parts that had none: 1
Changed lines of the file:
@@
 $EndComp
 $Comp
-L GNDREF #PWR01
+L GNDREF #PWR2
 U 1 1 5AB6F1A6
 P 3100 3200
-F 0 "#PWR01" H 3100 2950 50  0001 C CNN
+F 0 "#PWR2" H 3100 2950 50  0001 C CNN
 F 1 "GNDREF" H 3100 3050 50  0000 C CNN
 F 2 "" H 3100 3200 50  0001 C CNN
@@
 $EndComp
 $Comp
-L GNDREF #PWR02
+L GNDREF #PWR1
 U 1 1 5AB6F964
 P 2100 1550
-F 0 "#PWR02" H 2100 1300 50  0001 C CNN
+F 0 "#PWR1" H 2100 1300 50  0001 C CNN
 F 1 "GNDREF" H 2100 1400 50  0000 C CNN
 F 2 "" H 2100 1550 50  0001 C CNN
@@
 $EndComp
 $Comp
-L GNDREF #PWR03
+L GNDREF #PWR4
 U 1 1 5AB71FFB
 P 5150 1650
-F 0 "#PWR03" H 5150 1400 50  0001 C CNN
+F 0 "#PWR4" H 5150 1400 50  0001 C CNN
 F 1 "GNDREF" H 5150 1500 50  0000 C CNN
 F 2 "" H 5150 1650 50  0001 C CNN
@@
 $EndComp
 $Comp
-L GNDREF #PWR04
+L GNDREF #PWR3
 U 1 1 5AB975C6
 P 3150 4800
-F 0 "#PWR04" H 3150 4550 50  0001 C CNN
+F 0 "#PWR3" H 3150 4550 50  0001 C CNN
 F 1 "GNDREF" H 3150 4650 50  0000 C CNN
 F 2 "" H 3150 4800 50  0001 C CNN
@@
 $EndComp
 $Comp
-L GNDREF #PWR05
+L GNDREF #PWR7
 U 1 1 5AB981D8
 P 9350 5500
-F 0 "#PWR05" H 9350 5250 50  0001 C CNN
+F 0 "#PWR7" H 9350 5250 50  0001 C CNN
 F 1 "GNDREF" H 9350 5350 50  0000 C CNN
 F 2 "" H 9350 5500 50  0001 C CNN
@@
 $EndComp
 $Comp
-L GNDREF #PWR06
+L GNDREF #PWR5
 U 1 1 5AB98C16
 P 6100 3400
-F 0 "#PWR06" H 6100 3150 50  0001 C CNN
+F 0 "#PWR5" H 6100 3150 50  0001 C CNN
 F 1 "GNDREF" H 6100 3250 50  0000 C CNN
 F 2 "" H 6100 3400 50  0001 C CNN
@@
 $EndComp
 $Comp
-L GNDREF #PWR07
+L GNDREF #PWR6
 U 1 1 5AB98DC5
 P 9350 3850
-F 0 "#PWR07" H 9350 3600 50  0001 C CNN
+F 0 "#PWR6" H 9350 3600 50  0001 C CNN
 F 1 "GNDREF" H 9350 3700 50  0000 C CNN
 F 2 "" H 9350 3850 50  0001 C CNN
@@
 5V
 $Comp
-L R R?
+L R R29
 U 1 1 5ABCAE40
 P 8300 2150
-F 0 "R?" V 8380 2150 50  0000 C CNN
+F 0 "R29" V 8380 2150 50  0000 C CNN
 F 1 "R" V 8300 2150 50  0000 C CNN
 F 2 "" V 8230 2150 50  0001 C CNN
